File: mcu.kicad_sch (KiCad schematic)
At the start: 33 parts, among them SW1 SW_Nidec_CAS-120A1, SW2 SW_Push, U1 STM32H755ZIT6, Y1 25M, Y2 Crystal

Commit message: added load capacitors to oscillator
Parts:
- added C28, C29, C30, C31: 15p, symbol Device:C
Connections:
- net GND: now also C28.2, C29.2, C30.2, C31.2
- net HS_OSC_A: now also C28.1
- net HS_OSC_B: now also C29.1
- net LS_OSC_A: now also C31.1
- net LS_OSC_B: now also C30.1
