File: external.kicad_sch (KiCad schematic)
At the start: 0 parts

Commit message: Began external circuitry
Parts:
- added CN3: STE_I2C_QT, easyeda2kicad:CONN-SMD_BM04B-SRSS-TB, symbol CONN-SMD_BM04B-SRSS-TB:BM04B-SRSS-TB(LF)(SN)
- added F3, F4: Polyfuse, symbol Device:Polyfuse
- added M1, M2: Motor_Servo, symbol Motor:Motor_Servo
Connections:
- new net: F3.2, M1.2 (+)
- new net: F4.2, M2.2 (+)
- new net GND: CN3.0, CN3.1, M1.3 (-), M2.3 (-)
- new net NEOM9N.SCL: CN3.4
- new net NEOM9N.SDA: CN3.3
- new net SERVO PWM1: M1.1 (PWM)
- new net SERVO PWM2: M2.1 (PWM)
- new net VCC: CN3.2, F3.1, F4.1

Commit message: Current progress on externals
Other:
- note added: "To-do - Connect 2 Servo PWM channels -> DONE (from lawton) - Qwic connector with I2C peripheral -> DONE (from lawton) - SPI peripheral connector -> IN PROGRESS - Standard 0.1" header pinout - Transceiver output"
- note removed: "To-do - Connect 2 Servo PWM channels - Qwic connector with I2C peripheral - SPI peripheral connector"
Changed lines of the file:
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@@
 	(generator_version "9.0")
 	(paper "A4")
-	(text "To-do \n- Connect 2 Servo PWM channels \n- Qwic connector with I2C peripheral\n- SPI peripheral connector\n\n"
+	(text "To-do \n- Connect 2 Servo PWM channels \n	-> DONE (from lawton)\n- Qwic connector with I2C peripheral\n	-> DONE (from lawton)\n- SPI peripheral connector\n	-> IN PROGRESS\n- Standard 0.1\" header pinout\n- Transceiver output\n"
 		(exclude_from_sim no)
 		(at 123.444 88.138 0)
@@
 				(size 1.27 1.27)
 			)
+			(justify left)
 		)
 	)
