File: pwr.kicad_sch (KiCad schematic)
At the start: 26 parts, among them U10 STM32H755ZIT6

Commit message: some changes for 2027 aerolotl
Parts:
- removed C45: 220p, Capacitor_SMD:C_0402_1005Metric, symbol Device:C
- removed C48, C61, C64: 4.7u, Capacitor_SMD:C_0805_2012Metric, symbol Device:C
- removed C49: 10u, Capacitor_SMD:C_0805_2012Metric, symbol Device:C
- removed C50, C51, C52, C54, C55, C56, C57, C58, C59, C60, C62, C63, C65, C66, C67: 100n, Capacitor_SMD:C_0402_1005Metric, symbol Device:C
- removed C53, C68: 1u, Capacitor_SMD:C_0603_1608Metric, symbol Device:C
- removed FB3: 120, Inductor_SMD:L_0805_2012Metric, symbol Device:FerriteBead
- removed L4: 2.2u, Inductor_SMD:L_0805_2012Metric, symbol Device:L
- removed R48: 47, symbol Device:R
- removed U10: STM32H755ZIT6, Package_QFP:LQFP-144_20x20mm_P0.5mm, symbol MCU_ST_STM32H7:STM32H755ZITx
- added C1, C10, C11, C12, C13, C19, C2, C22, C3, C4, C5, C6, C7, C8, C9: 100n, symbol Device:C
- added C14, C16, C18: 4.7u, symbol Device:C
- added C15: 220p, symbol Device:C
- added C17: 10u, symbol Device:C
- added C20, C21, C23: 1u, symbol Device:C
- added FB1: 120, symbol Device:FerriteBead
- added L1: 2.2u, symbol Device:L
- added R1, R5: 10k, symbol Device:R
- added R3: 47, symbol Device:R
- added SW1: SW_Nidec_CAS-120A1, Button_Switch_SMD:Nidec_Copal_CAS-120A, symbol Switch:SW_Nidec_CAS-120A1
- added SW2: SW_Push, symbol Switch:SW_Push
- added U1: STM32H755ZIT6, Package_QFP:LQFP-144_20x20mm_P0.5mm, symbol MCU_ST_STM32H7:STM32H755ZITx
Connections:
- net +3.3VA: now also FB1.1, R3.1, U1.36 (VDDA)
- net +3V3: now also C1.1, C10.1, C11.1, C12.1, C13.1, C14.1, C16.1, C18.1, C19.1, C2.1, C20.1, C3.1, C4.1, C5.1, C6.1, C7.1, C8.1, C9.1, FB1.2, U1.105 (VDDLDO), U1.106 (VDD), U1.119 (VDD), U1.129 (VDD), U1.13 (VDD), U1.142 (PDR_ON), U1.143 (VDDLDO), U1.144 (VDD), U1.16 (VDDSMPS), U1.19 (VDD), U1.32 (VDD), U1.42 (VDD), U1.56 (VDD), U1.7 (VDD), U1.70 (VDDLDO), U1.71 (VDD), U1.79 (VDD), U1.8 (VBAT), U1.90 (VDD50_USB), U1.91 (VDD33_USB), U1.92 (VDD)
- net GND: now also C1.2, C10.2, C11.2, C12.2, C13.2, C14.2, C15.2, C16.2, C17.2, C18.2, C19.2, C2.2, C20.2, C21.2, C22.2, C23.2, C3.2, C4.2, C5.2, C6.2, C7.2, C8.2, C9.2, R5.2, SW2.1, U1.104 (VSS), U1.118 (VSS), U1.12 (VSS), U1.128 (VSS), U1.14 (VSSSMPS), U1.141 (VSS), U1.18 (VSS), U1.33 (VSS), U1.34 (VSSA), U1.41 (VSS), U1.55 (VSS), U1.6 (VSS), U1.69 (VSS), U1.80 (VSS), U1.89 (VSS)
- net VFBSMPS: now also C17.1, L1.2, U1.103 (VCAP), U1.140 (VCAP), U1.17 (VFBSMPS), U1.68 (VCAP)
- net VLX: now also C15.1, L1.1, U1.15 (VLXSMPS)
- new net: C22.1, C23.1, R3.2, U1.35 (VREF+)
- new net: C21.1, R1.2, SW2.2
- new net BOOT0: R5.1, SW1.2 (B), U1.135 (BOOT0)
- new net RESET: U1.27 (NRST)
- new net VCC: R1.1, SW1.3 (A)
