File: sheets/swd.kicad_sch (KiCad schematic)
At the start: 2 parts, among them J6 FTSH-107-STDC14

Commit message: polished up circuit, added new 16.8V to 7.4V step down circuit components
Connections:
- net GNDDetect: now reaches J6.11, R4.2
- net T_VCC renamed +3V3
Changed lines of the file:
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@@
-	(wire
-		(pts
-			(xy 115.57 93.98) (xy 121.92 93.98)
-		)
-		(stroke
-			(width 0)
-			(type default)
-		)
-	)
 	(wire
 		(pts
@@
 	(wire
 		(pts
+			(xy 113.03 89.535) (xy 113.03 93.98)
+		)
+		(stroke
+			(width 0)
+			(type default)
+		)
+	)
+	(wire
+		(pts
 			(xy 147.32 104.14) (xy 152.4 104.14)
 		)
@@
 	(wire
 		(pts
+			(xy 113.03 93.98) (xy 121.92 93.98)
+		)
+		(stroke
+			(width 0)
+			(type default)
+		)
+	)
+	(wire
+		(pts
 			(xy 87.63 104.14) (xy 87.63 107.95)
 		)
@@
 		)
 	)
-	(label "T_NRST"
-		(at 152.4 104.14 0)
-		(effects
-			(font
-				(size 1.27 1.27)
-			)
-			(justify left bottom)
-		)
-	)
-	(label "T_SWO"
-		(at 152.4 99.06 0)
+	(label "GNDDetect"
+		(at 110.49 104.14 0)
 		(effects
 			(font
@@
 		)
 	)
-	(label "T_SWDIO"
-		(at 152.4 93.98 0)
-		(effects
-			(font
-				(size 1.27 1.27)
-			)
-			(justify left bottom)
-		)
-	)
-	(label "T_SWCLK"
-		(at 152.4 96.52 0)
-		(effects
-			(font
-				(size 1.27 1.27)
-			)
-			(justify left bottom)
-		)
-	)
 	(label "T_VCC"
 		(at 115.57 93.98 0)
@@
 			)
 			(justify left bottom)
+		)
+	)
+	(hierarchical_label "T_SWCLK"
+		(shape output)
+		(at 152.4 96.52 0)
+		(effects
+			(font
+				(size 1.27 1.27)
+			)
+			(justify left)
+		)
+	)
+	(hierarchical_label "T_SWO"
+		(shape input)
+		(at 152.4 99.06 0)
+		(effects
+			(font
+				(size 1.27 1.27)
+			)
+			(justify left)
 		)
 	)
@@
 		(shape input)
 		(at 157.48 106.68 0)
+		(effects
+			(font
+				(size 1.27 1.27)
+			)
+			(justify left)
+		)
+	)
+	(hierarchical_label "T_SWDIO"
+		(shape bidirectional)
+		(at 152.4 93.98 0)
+		(effects
+			(font
+				(size 1.27 1.27)
+			)
+			(justify left)
+		)
+	)
+	(hierarchical_label "T_NRST"
+		(shape bidirectional)
+		(at 152.4 104.14 0)
 		(effects
 			(font
@@
 					(unit 1)
 				)
+			)
+		)
+	)
+	(symbol
+		(lib_id "power:+3V3")
+		(at 113.03 89.535 0)
+		(unit 1)
+		(exclude_from_sim no)
+		(in_bom yes)
+		(on_board yes)
+		(dnp no)
+		(fields_autoplaced yes)
+		(property "Reference" "#PWR068"
+			(at 113.03 93.345 0)
+			(effects
+				(font
+					(size 1.27 1.27)
+				)
+				(hide yes)
+			)
+		)
+		(property "Value" "+3V3"
+			(at 113.03 85.09 0)
+			(effects
+				(font
+					(size 1.27 1.27)
+				)
+			)
+		)
+		(property "Footprint" ""
+			(at 113.03 89.535 0)
+			(effects
+				(font
+					(size 1.27 1.27)
+				)
+				(hide yes)
+			)
+		)
+		(property "Datasheet" ""
+			(at 113.03 89.535 0)
+			(effects
+				(font
+					(size 1.27 1.27)
+				)
+				(hide yes)
+			)
+		)
+		(property "Description" "Power symbol creates a global label with name \"+3V3\""
+			(at 113.03 89.535 0)
+			(effects
+				(font
+					(size 1.27 1.27)
+				)
+				(hide yes)
+			)
+		)
+		(pin "1"
+		)
+		(instances
+			(project ""
+				(path "/3f5bc5ea-feaa-4ed9-b0e0-c918b1fb5754/226d91b5-727a-47f8-9cda-891697ac9edb"
+					(reference "#PWR068")
+					(unit 1)
+				)

Commit message: Rev1 schematic done
Parts:
- J1: renamed from J6; footprint aerolotl_custom:SAMTEC_FTSH-107-01-L-DV-K-A -> aerolotl_custom:STDC14_SAMTEC_FTSH-107-01-L-DV-K-A
Other:
- moved on the sheet: J1, R4
