File: sheets/swd.kicad_sch (KiCad schematic)
At the start: 2 parts, among them J1 FTSH-107-STDC14

Commit message: some changes for 2027 aerolotl
Changed lines of the file:
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@@
 	(wire
 		(pts
-			(xy 154.94 106.68) (xy 165.1 106.68)
+			(xy 154.94 106.68) (xy 160.02 106.68)
 		)
 		(stroke
@@
 	(hierarchical_label "T_VCP_RX"
 		(shape input)
-		(at 165.1 106.68 0)
+		(at 160.02 106.68 0)
 		(effects
 			(font
