File: pre-layout-backup/aerolotl.kicad_pcb (KiCad board)
At the start: 4 copper layers, 152.4 x 152.4 mm, 185 parts, among them CN1 StemmaQT, CN2 StemmaQT, J1 FTSH-107-STDC14, J10 USART3, J11 UART8, J13 GPIO_PE2-PE6, J14 Screw_Terminal_01x02, J16 GPIO_PE7-PE11, J17 Conn_01x05_Pin, J18 SERVO1, J19 SERVO2, J20 SREVO3, J21 SERVO4, J3 Pin Switch Conn, J4 USB_C_Receptacle_USB2.0_16P, J5 Screw_Terminal_01x02, J7 SPARE_ADC1, J8 Conn_01x04_Pin, Q1 AO3400A, Q4 AO4407A, Q5 FDS6673BZ_C467780, Q6 FDS6673BZ_C467780, Q7 AO3400A, Q8 AO3400A, SW1 SW_Push, SW2 SW_SPST, SW4 SW_SPST, U1 ADXL345BCCZ-RL7, U10 BMI088, U12 Airlift, U14 STM32H723VGTx, U2 USBLC6-2P6, U3 TPS2116DRL, U4 AMS1117-3.3, U5 LMR51430XFDDCR, U6 MAX-M10S, U7 BMP581, U9 ADXL375BCCZ-RL7, X1 X322525MOB4SI, Y3 32k768

Commit message: Save Aerolotl PCB and schematic progress
Parts:
- removed CN1, CN2: StemmaQT, aerolotl_custom:StemmaQT
- removed J4: USB_C_Receptacle_USB2.0_16P, Connector_USB:USB_C_Receptacle_HRO_TYPE-C-31-M-12
- removed U1: ADXL345BCCZ-RL7, aerolotl_custom:ADXL345
- moved J13 356.9 mm to (440.2, 54.5), turned to 0 degrees
- moved U12 348.9 mm to (442.2, 110.1)
- moved J17 347.3 mm to (427.0, 59.4), turned to 0 degrees
- moved J16 345.1 mm to (440.2, 62.2), turned to 0 degrees
- moved J8 342.0 mm to (438.3, 31.6), turned to 0 degrees
- moved J11 333.6 mm to (438.3, 46.9), turned to 0 degrees
- moved J10 324.2 mm to (438.3, 39.2), turned to 0 degrees
- moved C85 315.9 mm to (443.5, 98.9), turned to 0 degrees
- moved C47 315.9 mm to (433.6, 74.9)
- moved D11 314.1 mm to (439.2, 99.6)
- moved R5 313.9 mm to (441.4, 76.3), turned to 0 degrees
- moved C46 312.2 mm to (441.4, 71.3)
- moved Y3 311.4 mm to (435.4, 128.0), turned to 0 degrees
- moved TP9 310.0 mm to (425.2, 86.3)
- moved R46 309.8 mm to (442.2, 85.0)
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Routing:
- removed copper zone on In2.Cu, net +12V
- removed copper zone on In2.Cu, net +3V3
- removed copper zone on In1.Cu, net GND
Other:
- board text added: "RF (GPS antenna -> SAW -> RF_IN): net class RF 50 ohm coplanar waveguide (CPWG), L1 ref L2 GND Stackup JLC04161H-7628 (7628 prepreg 0.2104 mm, er~4.4) Width 0.306 mm (12.04 mil), gap to GND pour 0.203 mm (8 mil) Values from JLCPCB impedance calculator. Stitch GND vias both sides."
- board text added: "USB D+/D-: net class USB (diff pair) 90 ohm differential, non-coplanar, L1 ref L2 GND Stackup JLC04161H-7628 (7628 prepreg 0.2104 mm, er~4.4) Width 0.291 mm (11.44 mil), pair gap 0.203 mm (8 mil) Values from JLCPCB impedance calculator. Keep pour >=0.5 mm away."
- board text removed: "PLACE J4 (USB-C, after F8)"
