File: pre-layout-backup/external.kicad_sch (KiCad schematic)
At the start: 28 parts, among them CN1 StemmaQT, CN2 StemmaQT, J10 USART3, J11 UART8, J13 GPIO_PE2-PE6, J16 GPIO_PE7-PE11, J17 Conn_01x05_Pin, J18 SERVO1, J19 SERVO2, J20 SREVO3, J21 SERVO4, J7 SPARE_ADC1, J8 Conn_01x04_Pin

Commit message: Save Aerolotl PCB and schematic progress
Parts:
- CN1, CN2: footprint aerolotl_custom:StemmaQT -> aerolotl_custom:CONN-SMD_BM04B-SRSS-TB
Changed lines of the file:
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@@
 			)
 		)
-		(property "Footprint" "aerolotl_custom:StemmaQT"
+		(property "Footprint" "aerolotl_custom:CONN-SMD_BM04B-SRSS-TB"
 			(at 38.1 53.34 0)
 			(hide yes)
@@
 			)
 		)
-		(property "Footprint" "aerolotl_custom:StemmaQT"
+		(property "Footprint" "aerolotl_custom:CONN-SMD_BM04B-SRSS-TB"
 			(at 78.74 52.07 0)
 			(hide yes)
