File: pre-layout-backup/power.kicad_sch (KiCad schematic)
At the start: 38 parts, among them J3 Pin Switch Conn, J4 USB_C_Receptacle_USB2.0_16P, Q4 AO4407A, SW4 SW_SPST, U2 USBLC6-2P6, U3 TPS2116DRL, U4 AMS1117-3.3, U5 LMR51430XFDDCR

Commit message: Save Aerolotl PCB and schematic progress
Parts:
- J4: footprint Connector_USB:USB_C_Receptacle_HRO_TYPE-C-31-M-12 -> (none)
Changed lines of the file:
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@@
 			)
 		)
-		(property "Footprint" "Connector_USB:USB_C_Receptacle_HRO_TYPE-C-31-M-12"
+		(property "Footprint" ""
 			(at 41.91 60.96 0)
 			(hide yes)
