File: pre-layout-backup/sensors.kicad_sch (KiCad schematic)
At the start: 18 parts, among them U1 ADXL345BCCZ-RL7, U10 BMI088, U6 MAX-M10S, U7 BMP581, U9 ADXL375BCCZ-RL7

Commit message: Save Aerolotl PCB and schematic progress
Parts:
- U1: footprint aerolotl_custom:ADXL345 -> ADXL345BCCZ-RL7:PQFN80P500X300X100-14N
Changed lines of the file:
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@@
 			)
 		)
-		(property "Footprint" "aerolotl_custom:ADXL345"
+		(property "Footprint" "ADXL345BCCZ-RL7:PQFN80P500X300X100-14N"
 			(at 199.39 57.15 0)
 			(hide yes)
