File: pre-rev2-backup/aerolotl.kicad_sch (KiCad schematic)
At the start: 0 parts

Commit message: Save Aerolotl PCB and schematic progress
Other:
- sheet External ports: added GPIO{PORT_G}; removed GPIO{PORT_E}
- sheet MCU ports: added 7V4_P_GOOD, GPIO{PORT_G}, SPI2{SCK, MISO, MOSI}; removed GPS_RST, PWR_STS, SPI2{SCK, MISO, MOSI, CS, BUSY, RST}
- sheet Power ports: added 7V4_P_GOOD; removed none
- sheet Sensors ports: added T_NRST; removed GPS_RST
- sheet airlift ports: added SPI2{SCK, MISO, MOSI}; removed SPI2{SCK, MISO, MOSI, CS, BUSY, RST}
Changed lines of the file:
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@@
 		)
+	)
+	(junction
+		(at 111.76 107.95)
+		(diameter 0)
+		(color 0 0 0 0)
 	)
 	(bus_entry
@@
 	(wire
 		(pts
-			(xy 104.14 210.82) (xy 142.24 210.82)
+			(xy 111.76 210.82) (xy 111.76 107.95)
 		)
 		(stroke
@@
 	(wire
 		(pts
+			(xy 104.14 210.82) (xy 111.76 210.82)
+		)
+		(stroke
+			(width 0)
+			(type default)
+		)
+	)
+	(wire
+		(pts
 			(xy 113.03 105.41) (xy 134.62 105.41)
 		)
@@
 	(wire
 		(pts
-			(xy 142.24 210.82) (xy 142.24 177.8)
-		)
-		(stroke
-			(width 0)
-			(type default)
-		)
-	)
-	(wire
-		(pts
 			(xy 222.25 208.28) (xy 293.37 208.28)
 		)
@@
 	(wire
 		(pts
+			(xy 105.41 135.89) (xy 134.62 135.89)
+		)
+		(stroke
+			(width 0)
+			(type default)
+		)
+	)
+	(wire
+		(pts
 			(xy 276.86 92.71) (xy 276.86 57.15)
 		)
@@
 		(pts
 			(xy 127 91.44) (xy 134.62 91.44)
-		)
-		(stroke
-			(width 0)
-			(type default)
-		)
-	)
-	(wire
-		(pts
-			(xy 105.41 130.81) (xy 134.62 130.81)
 		)
 		(stroke
@@
 			)
 		)
-		(pin "SPI2{SCK, MISO, MOSI, CS, BUSY, RST}" bidirectional
+		(pin "SPI2{SCK, MISO, MOSI}" bidirectional
 			(at 200.66 217.17 90)
 			(effects
@@
 			)
 		)
-		(pin "GPIO{PORT_E}" bidirectional
+		(pin "GPIO{PORT_G}" bidirectional
 			(at 293.37 120.65 180)
 			(effects
@@
 			)
 		)
+		(pin "7V4_P_GOOD" output
+			(at 105.41 135.89 0)
+			(effects
+				(font
+					(size 1.27 1.27)
+				)
+				(justify right)
+			)
+		)
 		(pin "PWR_STS" output
 			(at 105.41 130.81 0)
@@
 			)
 		)
-		(pin "GPS_RST" input
+		(pin "T_NRST" bidirectional
 			(at 104.14 210.82 0)
 			(effects
@@
 			)
 		)
-		(pin "SPI2{SCK, MISO, MOSI, CS, BUSY, RST}" bidirectional
+		(pin "SPI2{SCK, MISO, MOSI}" bidirectional
 			(at 200.66 177.8 270)
 			(effects
@@
 			)
 		)
-		(pin "GPIO{PORT_E}" bidirectional
+		(pin "GPIO{PORT_G}" bidirectional
 			(at 250.19 120.65 0)
 			(effects
@@
 			)
 		)
+		(pin "7V4_P_GOOD" input
+			(at 134.62 135.89 180)
+			(effects
+				(font
+					(size 1.27 1.27)
+				)
+				(justify left)
+			)
+		)
+		(pin "GPIO{PORT_E}" bidirectional
+			(at 168.91 85.09 90)
+			(effects
+				(font
+					(size 1.27 1.27)
+				)
+				(justify right)
+			)
+		)
 		(pin "USB_D+" bidirectional
+			(at 134.62 121.92 180)
+			(effects
+				(font
+					(size 1.27 1.27)
+				)
+				(justify left)
+			)
+		)
+		(pin "USB_D-" bidirectional
 			(at 134.62 124.46 180)
-			(effects
-				(font
-					(size 1.27 1.27)
-				)
-				(justify left)
-			)
-		)
-		(pin "USB_D-" bidirectional
-			(at 134.62 121.92 180)
 			(effects
 				(font
@@
 			(effects
 				(font
-					(size 1.27 1.27)
-				)
-				(justify right)
-			)
-		)
-		(pin "PWR_STS" input
-			(at 134.62 130.81 180)
-			(effects
-				(font
-					(size 1.27 1.27)
-				)
-				(justify left)
-			)
-		)
-		(pin "GPS_RST" output
-			(at 142.24 177.8 270)
-			(effects
-				(font
