File: pre-rev2-backup/airlift.kicad_sch (KiCad schematic)
At the start: 1 part, among them U12 Airlift

Commit message: Save Aerolotl PCB and schematic progress
Parts:
- U12: footprint Connector_PinSocket_2.54mm:PinSocket_1x12_P2.54mm_Vertical -> (none)
Connections:
- net SPI2.BUSY: no longer names the net of U12.8 (BUSY)
- net SPI2.CS: no longer names the net of U12.7 (CS)
- net SPI2.RST: no longer names the net of U12.9 (~{RST})
Changed lines of the file:
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@@
-		)
-	)
-	(label "SPI2.BUSY"
-		(at 160.02 107.95 0)
-		(effects
-			(font
-				(size 1.27 1.27)
-			)
-			(justify left bottom)
-		)
-	)
-	(label "SPI2.CS"
-		(at 129.54 107.95 180)
-		(effects
-			(font
-				(size 1.27 1.27)
-			)
-			(justify right bottom)
 		)
 	)
@@
 			)
 			(justify left bottom)
-		)
-	)
-	(label "SPI2.RST"
-		(at 129.54 92.71 180)
-		(effects
-			(font
-				(size 1.27 1.27)
-			)
-			(justify right bottom)
 		)
 	)
@@
 		)
 	)
-	(hierarchical_label "SPI2{SCK, MISO, MOSI, CS, BUSY, RST}"
+	(hierarchical_label "SPI2{SCK, MISO, MOSI}"
 		(shape bidirectional)
 		(at 114.3 90.17 180)
@@
 			)
 		)
-		(property "Footprint" "Connector_PinSocket_2.54mm:PinSocket_1x12_P2.54mm_Vertical"
+		(property "Footprint" ""
 			(at 132.08 88.9 0)
 			(hide yes)
