File: pre-rev2-backup/sheets/igniter.kicad_sch (KiCad schematic)
At the start: 39 parts, among them J14 Screw_Terminal_01x02, J5 Screw_Terminal_01x02, Q5 FDS6673BZ_C467780, Q6 FDS6673BZ_C467780, Q7 AO3400A, Q8 AO3400A

Commit message: Save Aerolotl PCB and schematic progress
Parts:
- removed C85, C86: 100n, Capacitor_SMD:C_0402_1005Metric, symbol Device:C
- removed D11, D12: 1N4148W, Diode_SMD:D_SOD-123, symbol Device:D
- removed R68, R70, R71, R73: 10k, Resistor_SMD:R_0402_1005Metric, symbol Device:R
- removed R69, R72: 33k, Resistor_SMD:R_0402_1005Metric, symbol Device:R
- C46, C52: footprint Capacitor_SMD:C_0603_1608Metric -> (none)
- C47, C50: footprint Capacitor_SMD:CP_Elec_8x10 -> (none); symbol Device:C_Polarized -> Device:C
- D7, D8: footprint LED_SMD:LED_0603_1608Metric -> (none)
- J14, J5: footprint TerminalBlock_Phoenix:TerminalBlock_Phoenix_MKDS-1,5-2-5.08_1x02_P5.08mm_Horizontal -> Connector_PinHeader_2.54mm:PinHeader_1x02_P2.54mm_Vertical
- R39, R40, R42, R43, R44, R52: footprint Resistor_SMD:R_0402_1005Metric -> (none)
- R45, R46: footprint Resistor_SMD:R_1206_3216Metric -> (none)
- R5, R6: footprint Resistor_SMD:R_0603_1608Metric -> (none)
Connections:
- net +12V_ARM: now also C47.2, C50.2; no longer C47.1, C50.1
- net GND: now also C47.1, C50.1; no longer C47.2, C50.2
- net IGN0: no longer TP9.1
- net IGN1: no longer TP10.1
- net IGN0_HS: no longer names the net of J14.1 (Pin_1), Q5.5 (D), Q5.6 (D), Q5.7 (D), Q5.8 (D)
- net IGN1_HS: no longer names the net of J5.1 (Pin_1), Q6.5 (D), Q6.6 (D), Q6.7 (D), Q6.8 (D)
- new net IGNITE_0: TP9.1
- new net IGNITE_1: TP10.1
Other:
- note removed: "Bias ~0.3 mA from 3V3 (far below e-match no-fire). Open: ADC ~0.57 V E-match present: ~0 V Firing (12.6 V): ~2.9 V"
- note removed: "CH0 (Drogue)"
- note removed: "CH1 (Main)"
- note removed: "Continuity / fire sense (per channel)"
- moved on the sheet: F4
