File: pre-rev2-backup/sheets/indicators.kicad_sch (KiCad schematic)
At the start: 17 parts, among them Q1 AO3400A

Commit message: Save Aerolotl PCB and schematic progress
Parts:
- BZ1: footprint aerolotl_custom:BUZ-TH_BD9.0-P5.00-D0.6-FD -> (none)
- C44: footprint Capacitor_SMD:C_0805_2012Metric -> (none); LCSC Part C45783 -> (none)
- C49: footprint Capacitor_SMD:C_0402_1005Metric -> (none); LCSC Part C1525 -> (none)
- R19, R20, R21, R22, R23, R24, R25: footprint Resistor_SMD:R_0402_1005Metric -> (none)
- R27: footprint Resistor_SMD:R_0603_1608Metric -> (none)
Changed lines of the file:
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@@
 			)
 		)
-		(property "Footprint" "Resistor_SMD:R_0402_1005Metric"
+		(property "Footprint" ""
 			(at 62.23 61.468 90)
 			(hide yes)
@@
 			)
 		)
-		(property "Footprint" "Resistor_SMD:R_0402_1005Metric"
+		(property "Footprint" ""
 			(at 62.23 51.308 90)
 			(hide yes)
@@
 			)
 		)
-		(property "Footprint" "Resistor_SMD:R_0402_1005Metric"
+		(property "Footprint" ""
 			(at 36.322 128.27 90)
 			(hide yes)
@@
 			)
 		)
-		(property "Footprint" "Resistor_SMD:R_0402_1005Metric"
+		(property "Footprint" ""
 			(at 181.102 62.23 90)
 			(hide yes)
@@
 			)
 		)
-		(property "Footprint" "Resistor_SMD:R_0402_1005Metric"
+		(property "Footprint" ""
 			(at 215.392 62.23 90)
 			(hide yes)
@@
 			)
 		)
-		(property "Footprint" "Resistor_SMD:R_0603_1608Metric"
+		(property "Footprint" ""
 			(at 250.952 60.96 90)
 			(hide yes)
@@
 			)
 		)
-		(property "Footprint" "aerolotl_custom:BUZ-TH_BD9.0-P5.00-D0.6-FD"
+		(property "Footprint" ""
 			(at 52.705 107.95 90)
 			(hide yes)
@@
 			)
 		)
-		(property "Footprint" "Capacitor_SMD:C_0805_2012Metric"
+		(property "Footprint" ""
 			(at 84.7852 113.03 0)
 			(hide yes)
@@
 		)
 		(property "Description" "Unpolarized capacitor"
-			(at 83.82 109.22 0)
-			(hide yes)
-			(show_name no)
-			(do_not_autoplace no)
-			(effects
-				(font
-					(size 1.27 1.27)
-				)
-			)
-		)
-		(property "LCSC Part" "C45783"
 			(at 83.82 109.22 0)
 			(hide yes)
@@
 			)
 		)
-		(property "Footprint" "Resistor_SMD:R_0402_1005Metric"
+		(property "Footprint" ""
 			(at 148.082 63.5 90)
 			(hide yes)
@@
 			)
 		)
-		(property "Footprint" "Capacitor_SMD:C_0402_1005Metric"
+		(property "Footprint" ""
 			(at 72.0852 113.03 0)
 			(hide yes)
@@
 		)
 		(property "Description" "Unpolarized capacitor"
-			(at 71.12 109.22 0)
-			(hide yes)
-			(show_name no)
-			(do_not_autoplace no)
-			(effects
-				(font
-					(size 1.27 1.27)
-				)
-			)
-		)
-		(property "LCSC Part" "C1525"
 			(at 71.12 109.22 0)
 			(hide yes)
@@
 			)
 		)
-		(property "Footprint" "Resistor_SMD:R_0402_1005Metric"
+		(property "Footprint" ""
 			(at 62.23 56.388 90)
 			(hide yes)
