File: pre-rev2-backup/sheets/power.kicad_sch (KiCad schematic)
At the start: 38 parts, among them J3 Pin Switch Conn, J4 USB_C_Receptacle_USB2.0_16P, Q4 AO4407A, SW4 SW_SPST, U2 USBLC6-2P6, U3 TPS2116DRL, U4 AMS1117-3.3, U5 LMR51430XFDDCR

Commit message: Save Aerolotl PCB and schematic progress
Parts:
- removed J4: USB_C_Receptacle_USB2.0_16P, Connector_USB:USB_C_Receptacle_HRO_TYPE-C-31-M-12, symbol Connector:USB_C_Receptacle_USB2.0_16P
- added J2: USB_C_Receptacle_USB2.0_16P, symbol Connector:USB_C_Receptacle_USB2.0_16P
- C1, C41: footprint Capacitor_SMD:C_1206_3216Metric -> (none)
- C2, C3: footprint Capacitor_SMD:C_0402_1005Metric -> (none)
- C31, C34: footprint Capacitor_SMD:C_0805_2012Metric -> (none); LCSC Part C45783 -> (none)
- C37: footprint Capacitor_SMD:C_0805_2012Metric -> (none)
- C38, C39: footprint Capacitor_SMD:C_0603_1608Metric -> (none); LCSC Part C14663 -> (none)
- J3: footprint Connector_AMASS:AMASS_XT30PW-M_1x02_P2.50mm_Horizontal -> (none)
- L3: footprint Inductor_SMD:L_Sunlord_SWPA4030S -> (none)
- R1: footprint Resistor_SMD:R_0603_1608Metric -> (none)
- R10, R11, R14, R15, R16, R48, R8, R9: footprint Resistor_SMD:R_0402_1005Metric -> (none)
- R13, R7: footprint Resistor_SMD:R_0402_1005Metric -> (none); LCSC Part C25744 -> (none)
- SW4: footprint Connector_JST:JST_XH_B2B-XH-A_1x02_P2.50mm_Vertical -> (none)
Connections:
- net GND: now also J2.A1 (GND), J2.A12 (GND), J2.B1 (GND), J2.B12 (GND), J2.S1 (SHIELD)
- net P_VBUS: now also J2.A4 (VBUS), J2.A9 (VBUS), J2.B4 (VBUS), J2.B9 (VBUS)
- net USB_DM: now also J2.A7 (D-), J2.B7 (D-)
- net USB_DP: now also J2.A6 (D+), J2.B6 (D+)
- net at R8.1: now also J2.A5 (CC1)
- net at R9.1: now also J2.B5 (CC2)
Other:
- note added: "22 ohm termination"
- note removed: "USB D+/D- 90 ohm differential, non-coplanar, L1 ref L2 GND Stackup JLC04161H-7628 (7628 prepreg 0.2104 mm, er~4.4) Width 0.291 mm (11.44 mil), pair gap 0.203 mm (8 mil) Values from JLCPCB impedance calculator. Keep pour >=0.5 mm away."
