File: pre-rev2-backup/sheets/sensors.kicad_sch (KiCad schematic)
At the start: 18 parts, among them U1 ADXL345BCCZ-RL7, U10 BMI088, U6 MAX-M10S, U7 BMP581, U9 ADXL375BCCZ-RL7

Commit message: Save Aerolotl PCB and schematic progress
Parts:
- removed SAW2: B39162B4300F210, aerolotl_custom:FILTER-SMD_5P-L1.4-W1.1_RSFPXXXXD, symbol aerolotl_custom:B39162B4300F210
- removed U1: ADXL345BCCZ-RL7, aerolotl_custom:ADXL345, symbol aerolotl_custom:ADXL345BCCZ-RL7
- added SAW1: B39162B4300F210, aerolotl_custom:FILTER-SMD_5P-L1.4-W1.1_RSFPXXXXD, symbol aerolotl_custom:B39162B4300F210
- added U8: ADXL345BCCZ-RL7, aerolotl_custom:ADXL345, symbol aerolotl_custom:ADXL345BCCZ-RL7
- AE1: footprint ANT_GP.1575.18.4.A.02_TAL -> aerolotl_custom:ANT_GP.1575.18.4.A.02_TAL
- C42, C43, C45, C48, CIO2, CS1: footprint Capacitor_SMD:C_0402_1005Metric -> (none); LCSC Part C1525 -> (none)
- CIO1, CS2: footprint Capacitor_SMD:C_0402_1005Metric -> (none)
- R17, R18, R47: footprint Resistor_SMD:R_0402_1005Metric -> (none)
Connections:
- net +3V3: now also U8.1 (VDD_I/O), U8.3 (RESERVED_3)
- net GND: now also SAW1.2 (GND), SAW1.3 (GND), SAW1.5 (GND), U8.11 (RESERVED_11), U8.2 (GND), U8.4 (GND), U8.5 (GND)
- net SPI1.CS_345: now also U8.7 (~{CS})
- net SPI1.INT_345: now also U8.8 (INT1)
- net SPI1.MISO: now also U8.12 (SDO/ALT_ADDRESS)
- net SPI1.MOSI: now also U8.13 (SDA/SDI/SDIO)
- net SPI1.SCK: now also U8.14 (SCL/SCLK)
- net at AE1.1: now also SAW1.1 (IN)
- net at CS2.1, R47.2: now also U8.6 (VS)
- net GPS_RF_IN: no longer names the net of U6.11 (RF_IN)
- net GPS_RF_IN: now also SAW1.4 (OUT)
- net GPS_RST renamed T_NRST
Other:
- note removed: "RF (GPS antenna -> SAW -> RF_IN): net class RF 50 ohm CPWG, L1 ref L2 GND Stackup JLC04161H-7628 (7628 prepreg 0.2104 mm, er~4.4) Width 0.306 mm (12.04 mil), gap to GND pour 0.203 mm (8 mil) Stitch GND vias both sides."
