File: pre-rev2-backup/sheets/swd.kicad_sch (KiCad schematic)
At the start: 2 parts, among them J1 FTSH-107-STDC14

Commit message: Save Aerolotl PCB and schematic progress
Parts:
- R4: footprint Resistor_SMD:R_0402_1005Metric -> (none)
Changed lines of the file:
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@@
 			)
 		)
-		(property "Footprint" "Resistor_SMD:R_0402_1005Metric"
+		(property "Footprint" ""
 			(at 102.87 105.918 90)
 			(hide yes)
