File: pre-servo-backup/external.kicad_sch (KiCad schematic)
At the start: 28 parts, among them CN1 StemmaQT, CN2 StemmaQT, J10 USART3, J11 UART8, J13 GPIO_PE2-PE6, J16 GPIO_PE7-PE11, J17 Conn_01x05_Pin, J18 SERVO1, J19 SERVO2, J20 SREVO3, J21 SERVO4, J7 SPARE_ADC1, J8 Conn_01x04_Pin

Commit message: Save Aerolotl PCB and schematic progress
Parts:
- removed C77, C79, C81, C83: 100u 25V, Capacitor_SMD:CP_Elec_6.3x7.7, symbol Device:C_Polarized
- removed C78, C80, C82, C84: 100n 50V, Capacitor_SMD:C_0603_1608Metric, symbol Device:C
- removed D10: PESD5V0S1BA, Diode_SMD:D_SOD-323, symbol Device:D_TVS
- removed F10, F7, F8, F9: 1812L300/24SLER, Fuse:Fuse_1812_4532Metric, symbol aerolotl_custom:1812L300_24SLER
- removed J13: GPIO_PE2-PE6, Connector_JST:JST_GH_BM07B-GHS-TBT_1x07-1MP_P1.25mm_Vertical, symbol Connector:Conn_01x07_Pin
- removed J16: GPIO_PE7-PE11, Connector_JST:JST_GH_BM07B-GHS-TBT_1x07-1MP_P1.25mm_Vertical, symbol Connector:Conn_01x07_Pin
- removed J18: SERVO1, Connector_Molex:Molex_SPOX_5267-03A_1x03_P2.50mm_Vertical, symbol Connector:Conn_01x03_Pin
- removed J19: SERVO2, Connector_Molex:Molex_SPOX_5267-03A_1x03_P2.50mm_Vertical, symbol Connector:Conn_01x03_Pin
- removed J20: SREVO3, Connector_Molex:Molex_SPOX_5267-03A_1x03_P2.50mm_Vertical, symbol Connector:Conn_01x03_Pin
- removed J21: SERVO4, Connector_Molex:Molex_SPOX_5267-03A_1x03_P2.50mm_Vertical, symbol Connector:Conn_01x03_Pin
- removed R66: 4.7k, Resistor_SMD:R_0402_1005Metric, symbol Device:R
- removed R67: 330, Resistor_SMD:R_0402_1005Metric, symbol Device:R
- added C54: 100n, symbol Device:C
- added F1, F2, F5, F6: 1812L300/24SLER, Capacitor_SMD:C_0402_1005Metric, symbol aerolotl_custom:1812L300_24SLER
- added J12, J15, J6, J9: Conn_01x03_Pin, symbol Connector:Conn_01x03_Pin
- added J13, J16: Conn_01x06_Pin, symbol Connector:Conn_01x06_Pin
- added R41, R55, R58, R63: GX2512-2W-30MR-1%, aerolotl_custom:RES-SMD_L6.4-W3.2-1, symbol aerolotl_custom:GX2512-2W-30MR-1%
- added R53, R57, R60, R62: 15k, symbol Device:R
- added R54, R56, R59, R61: 1k, symbol Device:R
- added U11: MCP6004T-I/SL, aerolotl_custom:SOIC-14_L8.7-W3.9-P1.27-LS6.0-BL, symbol aerolotl_custom:MCP6004T-I_SL
- CN1, CN2: footprint aerolotl_custom:StemmaQT -> aerolotl_custom:CONN-SMD_BM04B-SRSS-TB
- J10, J11, J8: footprint Connector_JST:JST_GH_BM04B-GHS-TBT_1x04-1MP_P1.25mm_Vertical -> (none)
- J17: footprint Connector_JST:JST_GH_BM05B-GHS-TBT_1x05-1MP_P1.25mm_Vertical -> (none)
- J7: footprint Connector_JST:JST_GH_BM03B-GHS-TBT_1x03-1MP_P1.25mm_Vertical -> (none)
Connections:
- net +3V3: now also C54.1, J13.6 (Pin_6), J16.6 (Pin_6), U11.4 (VDD)
- net GND: now also C54.2, J13.1 (Pin_1), J16.1 (Pin_1), R41.1, R54.2, R55.1, R56.2, R58.1, R59.2, R61.2, R63.1, U11.11 (VSS)
- new net: F5.1, J6.2 (Pin_2)
- new net: J15.1 (Pin_1), R58.2, U11.12 (VIND+)
- new net: R59.1, R60.1, U11.13 (VIND-)
- new net: R56.1, R57.1, U11.6 (VINB-)
- new net: F1.1, J12.2 (Pin_2)
- new net: F2.1, J15.2 (Pin_2)
- new net: J9.1 (Pin_1), R63.2, U11.10 (VINC+)
- new net: R53.1, R54.1, U11.2 (VINA-)
- new net: J12.1 (Pin_1), R41.2, U11.3 (VINA+)
- new net: J6.1 (Pin_1), R55.2, U11.5 (VINB+)
- new net: R61.1, R62.1, U11.9 (VINC-)
- new net: F6.1, J9.2 (Pin_2)
- new net +7V4_SERVO: F1.2, F2.2, F5.2, F6.2
- new net GPIO.PG10_IO: J13.2 (Pin_2)
- new net GPIO.PG11_IO: J16.5 (Pin_5)
- new net GPIO.PG12_IO: J16.4 (Pin_4)
- new net GPIO.PG13_IO: J16.3 (Pin_3)
- new net GPIO.PG14_IO: J16.2 (Pin_2)
- new net GPIO.PG7_IO: J13.5 (Pin_5)
- new net GPIO.PG8_IO: J13.4 (Pin_4)
- new net GPIO.PG9_IO: J13.3 (Pin_3)
- new net SERVO1_SENSE: R53.2, U11.1 (VOUTA)
- new net SERVO2_SENSE: R60.2, U11.14 (VOUTD)
- new net SERVO3_SENSE: R57.2, U11.7 (VOUTB)
- new net SERVO4_SENSE: R62.2, U11.8 (VOUTC)
- new net SERVO_PWM1: J12.3 (Pin_3)
- new net SERVO_PWM2: J15.3 (Pin_3)
- new net SERVO_PWM3: J6.3 (Pin_3)
- new net SERVO_PWM4: J9.3 (Pin_3)
Other:
- note added: "Current Sensing included"
- note removed: "Half-duplex servo bus (single-wire UART)"
- note removed: "MCU: SERVO_UART -> PD1 = UART4_TX (AF8), single-wire half-duplex (HDSEL=1)"
- note removed: "PE2-PE11 general purpose I/O (3.3 V, 5 V-tolerant FT pins)"
- note removed: "Servo port 1"
- note removed: "Servo port 2"
- note removed: "Servo port 3"
- note removed: "Servo port 4"
