File: pre-servo-backup/mcu.kicad_sch (KiCad schematic)
At the start: 30 parts, among them SW1 SW_Push, SW2 SW_SPST, U14 STM32H723VGTx, X1 X322525MOB4SI, Y3 32k768

Commit message: Save Aerolotl PCB and schematic progress
Parts:
- removed H1, H2: MountingHole, MountingHole:MountingHole_6.4mm_M6_ISO7380, symbol Mechanical:MountingHole
- added C23, C25, C26, C27: 15p, Capacitor_SMD:C_0402_1005Metric, symbol Device:C
- added H1, H2: MountingHole_Pad, symbol Mechanical:MountingHole_Pad
- added U1: STM32H755ZIT6, Package_QFP:LQFP-144_20x20mm_P0.5mm, symbol MCU_ST_STM32H7:STM32H755ZITx
- added X2: X322525MOB4SI, aerolotl_custom:CRYSTAL-SMD_4P-L3.2-W2.5-BL, symbol aerolotl_custom:X322525MOB4SI
- added Y2: 32k768, Crystal:Crystal_SMD_3215-2Pin_3.2x1.5mm, symbol Device:Crystal
- C24: value 100n -> 1u
- R65: footprint Resistor_SMD:R_0402_1005Metric -> (none)
- SW1, SW2: footprint Button_Switch_SMD:SW_SPST_TL3342 -> (none)
Connections:
- net BOOT0: now also U1.135 (BOOT0)
- net BUZZER_PWM: now also U14.34 (PB0), U1.97 (PA8)
- net GND: now also C23.2, C25.2, C26.2, C27.2, H1.1, H2.1, X2.2 (GND), X2.4 (GND)
- net HS_OSC_A: now also C23.1, U1.25 (PH0), X2.1 (OSC1)
- net HS_OSC_B: now also C25.1, U1.26 (PH1), X2.3 (OSC2)
- net I2C1.SCL: now also U1.133 (PB6)
- net I2C1.SDA: now also U1.134 (PB7)
- net I2C2.SCL: now also U1.66 (PB10)
- net I2C2.SDA: now also U1.67 (PB11)
- net I2C4.SCL: now also U1.82 (PD12); no longer U14.59 (PD12)
- net I2C4.SDA: now also U1.83 (PD13); no longer U14.60 (PD13)
- net LED_B: now also U1.108 (PA15)
- net LED_G: now also U1.132 (PB5)
- net LED_R: now also U1.131 (PB4)
- net LS_OSC_A: now also C27.1, U1.10 (PC14), Y2.2
- net LS_OSC_B: now also C26.1, U1.11 (PC15), Y2.1
- net SDMMC1.CK: now also U1.111 (PC12)
- net SDMMC1.CMD: now also U1.114 (PD2)
- net SDMMC1.D0: now also U1.95 (PC8)
- net SDMMC1.D1: now also U1.96 (PC9)
- net SDMMC1.D2: now also U1.109 (PC10)
- net SDMMC1.D3: now also U1.110 (PC11)
- net SENSE_I0: now also U1.49 (PB0); no longer U14.22 (PA0)
- net SENSE_I1: now also U1.50 (PB1); no longer U14.23 (PA1)
- net SPARE_ADC1: now also U1.43 (PA4); no longer U14.28 (PA4)
- net SPI1.CS_345: now also U1.84 (PD14); no longer U14.87 (PD6)
- net SPI1.CS_375: now also U1.85 (PD15); no longer U14.88 (PD7)
- net SPI1.CS_BMP: now also U1.81 (PD11); no longer U14.86 (PD5)
- net SPI1.INT_345: now also U1.2 (PE3); no longer U14.64 (PC7)
- net SPI1.INT_375: now also U1.3 (PE4); no longer U14.95 (PB8)
- net SPI1.INT_BMP: now also U1.4 (PE5); no longer U14.96 (PB9)
- net SPI1.INT_IMU_ACC: now also U1.60 (PE10); no longer U14.45 (PE15)
- net SPI1.INT_IMU_GYRO: now also U1.61 (PE11); no longer U14.36 (PB2)
- net SPI1.MISO: now also U1.45 (PA6)
- net SPI1.MOSI: now also U1.46 (PA7)
- net SPI1.SCK: now also U1.44 (PA5)
- net SPI2.MISO: now also U1.74 (PB14)
- net SPI2.MOSI: now also U1.75 (PB15)
- net SPI2.SCK: now also U1.73 (PB13)
- net SPI4.MISO: now also U1.63 (PE13)
- net SPI4.MOSI: now also U1.64 (PE14)
- net SPI4.SCK: now also U1.62 (PE12)
- net SWCLK: now also U1.107 (PA14)
- net SWDIO: now also U1.102 (PA13)
- net SWO: now also U1.130 (PB3)
- net T_NRST: now also U1.27 (NRST)
- net UART8_RX: now also U1.138 (PE0)
- net UART8_TX: now also U1.139 (PE1)
- net USART1_RX: now also U1.99 (PA10)
- net USART1_TX: now also U1.98 (PA9)
- net USART2_RX: now also U1.40 (PA3)
- net USART2_TX: now also U1.39 (PA2)
- net USART3_RX: now also U1.77 (PD9)
- net USART3_TX: now also U1.76 (PD8)
- net VOLT_SENSE: now also U1.30 (PC2_C); no longer U14.15 (PC0)
- net GPIO.PE10: no longer names the net of U14.40 (PE10)
- net GPIO.PE11: no longer names the net of U14.41 (PE11)
- net GPIO.PE3: no longer names the net of U14.2 (PE3)
- net GPIO.PE4: no longer names the net of U14.3 (PE4)
- net GPIO.PE5: no longer names the net of U14.4 (PE5)
- net GPIO.PE6: no longer names the net of U14.5 (PE6)
- net GPIO.PE7: no longer names the net of U14.37 (PE7)
- net GPIO.PE8: no longer names the net of U14.38 (PE8)
- net GPIO.PE9: no longer names the net of U14.39 (PE9)
- net GPS_RST: no longer names the net of U14.91 (PB5)
- net PWR_STS: no longer names the net of U14.16 (PC1)
- net SERVO_UART: no longer names the net of U14.82 (PD1)
- net SPI1.CS_IMU_ACC: no longer names the net of U14.84 (PD3)
- net SPI1.CS_IMU_GYRO: no longer names the net of U14.85 (PD4)
- net SPI2.BUSY: no longer names the net of U14.57 (PD10)
- net SPI2.CS: no longer names the net of U14.51 (PB12)
- net SPI2.RST: no longer names the net of U14.58 (PD11)
- new net GPIO.PG10_IO: U1.123 (PG10)
- new net GPIO.PG11_IO: U1.124 (PG11)
- new net GPIO.PG12_IO: U1.125 (PG12)
- new net GPIO.PG13_IO: U1.126 (PG13)
- new net GPIO.PG14_IO: U1.127 (PG14)
- new net GPIO.PG7_IO: U1.87 (PG7)
- new net GPIO.PG8_IO: U1.88 (PG8)
- new net GPIO.PG9_IO: U1.122 (PG9)
- new net IGNITE_0: U1.58 (PE8)
- new net IGNITE_1: U1.59 (PE9)
- new net LED: U1.86 (PG6)
- new net SERVO1_SENSE: U1.37 (PA0)
- new net SERVO2_SENSE: U1.38 (PA1)
- new net SERVO_PWM1: U1.93 (PC6)
- new net SERVO_PWM2: U1.94 (PC7)
- new net SERVO_PWM3: U1.5 (PE6)
- new net SERVO_PWM4: U1.57 (PE7)
- new net USB_D_M: U1.100 (PA11)
- new net USB_D_P: U1.101 (PA12)
- no-connect marks 7 -> 27
Other:
- note added: "spi1 usart2 spare_adc1 buzzer_pwm usart1 usb swd led{r, g, b} i2c1 i2c2 spi2 sdmmc usart3 hs_osc gpio ports uart8 ignite_bus spi4"
