File: pre-stackup-backup/sheets/power.kicad_sch (KiCad schematic)
At the start: 38 parts, among them J3 Pin Switch Conn, J4 USB_C_Receptacle_USB2.0_16P, Q4 AO4407A, SW4 SW_SPST, U2 USBLC6-2P6, U3 TPS2116DRL, U4 AMS1117-3.3, U5 LMR51430XFDDCR

Commit message: Save Aerolotl PCB and schematic progress
Parts:
- removed J4: USB_C_Receptacle_USB2.0_16P, Connector_USB:USB_C_Receptacle_HRO_TYPE-C-31-M-12, symbol Connector:USB_C_Receptacle_USB2.0_16P
- added J2: USB_C_Receptacle_USB2.0_16P, Connector_USB:USB_C_Receptacle_HRO_TYPE-C-31-M-12, symbol Connector:USB_C_Receptacle_USB2.0_16P
Connections:
- net GND: now also J2.A1 (GND), J2.A12 (GND), J2.B1 (GND), J2.B12 (GND), J2.S1 (SHIELD)
- net P_VBUS: now also J2.A4 (VBUS), J2.A9 (VBUS), J2.B4 (VBUS), J2.B9 (VBUS)
- net USB_DM: now also J2.A7 (D-), J2.B7 (D-)
- net USB_DP: now also J2.A6 (D+), J2.B6 (D+)
- net at R8.1: now also J2.A5 (CC1)
- net at R9.1: now also J2.B5 (CC2)
Other:
- note added: "22 ohm termination"
- note removed: "USB D+/D- 90 ohm differential, non-coplanar, L1 ref L2 GND Stackup JLC04161H-7628 (7628 prepreg 0.2104 mm, er~4.4) Width 0.291 mm (11.44 mil), pair gap 0.203 mm (8 mil) Values from JLCPCB impedance calculator. Keep pour >=0.5 mm away."
Changed lines of the file:
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@@
 		)
 	)
-	(text "UVLO rising: 4.5V\nUVLO falling: 3.35V"
+	(text "22 ohm termination"
 		(exclude_from_sim no)
-		(at 186.69 24.13 0)
+		(at 107.95 66.04 0)
 		(effects
 			(font
@@
 		)
 	)
-	(text "Min Vin = Vout + 1.3V"
+	(text "UVLO rising: 4.5V\nUVLO falling: 3.35V"
 		(exclude_from_sim no)
-		(at 105.41 34.29 0)
+		(at 186.69 24.13 0)
 		(effects
 			(font
@@
 		)
 	)
-	(text "USB D+/D-\n90 ohm differential, non-coplanar, L1 ref L2 GND\n\nStackup JLC04161H-7628 (7628 prepreg 0.2104 mm, er~4.4)\nWidth 0.291 mm (11.44 mil), pair gap 0.203 mm (8 mil)\n\nValues from JLCPCB impedance calculator. Keep pour >=0.5 mm away."
+	(text "Min Vin = Vout + 1.3V"
 		(exclude_from_sim no)
-		(at 27.94 105.41 0)
+		(at 105.41 34.29 0)
 		(effects
 			(font
 				(size 1.27 1.27)
 			)
-			(justify left)
 		)
 	)
@@
 	)
 	(symbol
-		(lib_name "USB_C_Receptacle_USB2.0_16P_1")
-		(lib_id "Connector:USB_C_Receptacle_USB2.0_16P")
-		(at 38.1 60.96 0)
-		(unit 1)
-		(body_style 1)
-		(exclude_from_sim no)
-		(in_bom yes)
-		(on_board yes)
-		(in_pos_files yes)
-		(dnp no)
-		(fields_autoplaced yes)
-		(property "Reference" "J4"
-			(at 38.1 38.1 0)
-			(show_name no)
-			(do_not_autoplace no)
-			(effects
-				(font
-					(size 1.27 1.27)
-				)
-			)
-		)
-		(property "Value" "USB_C_Receptacle_USB2.0_16P"
-			(at 38.1 40.64 0)
-			(show_name no)
-			(do_not_autoplace no)
-			(effects
-				(font
-					(size 1.27 1.27)
-				)
-			)
-		)
-		(property "Footprint" "Connector_USB:USB_C_Receptacle_HRO_TYPE-C-31-M-12"
-			(at 41.91 60.96 0)
-			(hide yes)
-			(show_name no)
-			(do_not_autoplace no)
-			(effects
-				(font
-					(size 1.27 1.27)
-				)
-			)
-		)
-		(property "Datasheet" "https://www.usb.org/sites/default/files/documents/usb_type-c.zip"
-			(at 41.91 60.96 0)
-			(hide yes)
-			(show_name no)
-			(do_not_autoplace no)
-			(effects
-				(font
-					(size 1.27 1.27)
-				)
-			)
-		)
-		(property "Description" "USB 2.0-only 16P Type-C Receptacle connector"
-			(at 38.1 60.96 0)
-			(hide yes)
-			(show_name no)
-			(do_not_autoplace no)
-			(effects
-				(font
-					(size 1.27 1.27)
-				)
-			)
-		)
-		(pin "B4"
-		)
-		(pin "B5"
-		)
-		(pin "B1"
-		)
-		(pin "B7"
-		)
-		(pin "B6"
-		)
-		(pin "B9"
-		)
-		(pin "B8"
-		)
-		(pin "SH"
-		)
-		(pin "B12"
-		)
-		(pin "A7"
-		)
-		(pin "A12"
-		)
-		(pin "A6"
-		)
-		(pin "A9"
-		)
-		(pin "A8"
-		)
-		(pin "A1"
-		)
-		(pin "A4"
-		)
-		(pin "A5"
-		)
-		(instances
-			(project "aerolotl"
-				(path "/3f5bc5ea-feaa-4ed9-b0e0-c918b1fb5754/74cb3ba4-5441-4040-b144-f529fa281743"
-					(reference "J4")
-					(unit 1)
-				)
-			)
-		)
-	)
-	(symbol
 		(lib_id "Device:C")
 		(at 168.91 101.6 0)
@@
 					(unit 1)
 				)
+			)
+		)
+	)
+	(symbol
+		(lib_id "Connector:USB_C_Receptacle_USB2.0_16P")
+		(at 38.1 60.96 0)
+		(unit 1)
+		(body_style 1)
+		(exclude_from_sim no)
+		(in_bom yes)
+		(on_board yes)
+		(in_pos_files yes)
+		(dnp no)
+		(fields_autoplaced yes)
+		(property "Reference" "J2"
+			(at 38.1 38.1 0)
+			(show_name no)
+			(do_not_autoplace no)
+			(effects
+				(font
+					(size 1.27 1.27)
+				)
+			)
+		)
+		(property "Value" "USB_C_Receptacle_USB2.0_16P"
+			(at 38.1 40.64 0)
+			(show_name no)
+			(do_not_autoplace no)
+			(effects
+				(font
+					(size 1.27 1.27)
+				)
+			)
+		)
+		(property "Footprint" "Connector_USB:USB_C_Receptacle_HRO_TYPE-C-31-M-12"
+			(at 41.91 60.96 0)
+			(hide yes)
+			(show_name no)
+			(do_not_autoplace no)
+			(effects
+				(font
+					(size 1.27 1.27)
+				)
+			)
+		)
+		(property "Datasheet" "https://www.usb.org/sites/default/files/documents/usb_type-c.zip"
+			(at 41.91 60.96 0)
+			(hide yes)
+			(show_name no)
+			(do_not_autoplace no)
+			(effects
+				(font
+					(size 1.27 1.27)
+				)
+			)
+		)
+		(property "Description" "USB 2.0-only 16P Type-C Receptacle connector"
+			(at 38.1 60.96 0)
+			(hide yes)
+			(show_name no)
+			(do_not_autoplace no)
+			(effects
+				(font
+					(size 1.27 1.27)
+				)
+			)
+		)
+		(property "Dielectric" ""
+			(at 38.1 60.96 0)
+			(hide yes)
+			(show_name no)
+			(do_not_autoplace no)
+			(effects
+				(font
+					(size 1.27 1.27)
+				)
+			)
+		)
+		(property "Purchase-URL" ""
+			(at 38.1 60.96 0)
+			(hide yes)
+			(show_name no)
+			(do_not_autoplace no)
+			(effects
+				(font
+					(size 1.27 1.27)
+				)
+			)
+		)
+		(property "Tolerance" ""
+			(at 38.1 60.96 0)
+			(hide yes)
+			(show_name no)
+			(do_not_autoplace no)
+			(effects
+				(font
+					(size 1.27 1.27)
+				)
+			)
+		)
+		(property "Voltage" ""
+			(at 38.1 60.96 0)
+			(hide yes)
+			(show_name no)
+			(do_not_autoplace no)
+			(effects
+				(font
+					(size 1.27 1.27)
+				)
+			)
+		)
+		(pin "B8"
+		)
+		(pin "A7"
+		)
+		(pin "S1"
+		)
+		(pin "A1"
+		)
+		(pin "A8"
+		)
+		(pin "A5"
+		)
+		(pin "A12"
+		)
+		(pin "B1"
+		)
+		(pin "A4"
+		)
+		(pin "B12"
+		)
+		(pin "A6"
+		)
+		(pin "B6"
+		)
+		(pin "B7"
+		)
+		(pin "B5"
+		)
+		(pin "B9"
+		)
+		(pin "A9"
+		)
+		(pin "B4"
+		)
+		(instances
+			(project "aerolotl"
+				(path "/3f5bc5ea-feaa-4ed9-b0e0-c918b1fb5754/74cb3ba4-5441-4040-b144-f529fa281743"
+					(reference "J2")
+					(unit 1)
+				)
