File: pre-stackup-backup/sheets/sensors.kicad_sch (KiCad schematic)
At the start: 18 parts, among them U1 ADXL345BCCZ-RL7, U10 BMI088, U6 MAX-M10S, U7 BMP581, U9 ADXL375BCCZ-RL7

Commit message: Save Aerolotl PCB and schematic progress
Parts:
- removed SAW2: B39162B4300F210, aerolotl_custom:FILTER-SMD_5P-L1.4-W1.1_RSFPXXXXD, symbol aerolotl_custom:B39162B4300F210
- added SAW1: B39162B4300F210, aerolotl_custom:FILTER-SMD_5P-L1.4-W1.1_RSFPXXXXD, symbol aerolotl_custom:B39162B4300F210
- AE1: footprint ANT_GP.1575.18.4.A.02_TAL -> aerolotl_custom:ANT_GP.1575.18.4.A.02_TAL
- U1: footprint aerolotl_custom:ADXL345 -> ADXL345BCCZ-RL7:PQFN80P500X300X100-14N
Connections:
- net GND: now also SAW1.2 (GND), SAW1.3 (GND), SAW1.5 (GND)
- net at AE1.1: now also SAW1.1 (IN)
- net GPS_RF_IN: no longer names the net of U6.11 (RF_IN)
- net GPS_RF_IN: now also SAW1.4 (OUT)
Other:
- note removed: "RF (GPS antenna -> SAW -> RF_IN): net class RF 50 ohm CPWG, L1 ref L2 GND Stackup JLC04161H-7628 (7628 prepreg 0.2104 mm, er~4.4) Width 0.306 mm (12.04 mil), gap to GND pour 0.203 mm (8 mil) Stitch GND vias both sides."
Changed lines of the file:
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@@
 		)
 	)
-	(text "RF (GPS antenna -> SAW -> RF_IN): net class RF\n50 ohm CPWG, L1 ref L2 GND\n\nStackup JLC04161H-7628 (7628 prepreg 0.2104 mm, er~4.4)\nWidth 0.306 mm (12.04 mil), gap to GND pour 0.203 mm (8 mil)\n\nStitch GND vias both sides."
-		(exclude_from_sim no)
-		(at 81.28 137.16 0)
-		(effects
-			(font
-				(size 1.27 1.27)
-			)
-			(justify left)
-		)
-	)
 	(text "ADXL375"
 		(exclude_from_sim no)
@@
 		)
 	)
+	(text "netclass with impedance matching"
+		(exclude_from_sim no)
+		(at 120.65 128.27 0)
+		(effects
+			(font
+				(size 1.27 1.27)
+			)
+		)
+	)
 	(text "BMP581"
 		(exclude_from_sim no)
@@
 		)
 	)
-	(label "GPS_RF_IN"
-		(at 101.6 119.38 0)
-		(effects
-			(font
-				(size 1.27 1.27)
-			)
-			(justify left bottom)
-		)
-	)
 	(label "SPI1.CS_375"
 		(at 246.38 160.02 0)
@@
 	)
 	(symbol
-		(lib_id "aerolotl_custom:B39162B4300F210")
-		(at 115.57 107.95 0)
-		(unit 1)
-		(body_style 1)
-		(exclude_from_sim no)
-		(in_bom yes)
-		(on_board yes)
-		(in_pos_files yes)
-		(dnp no)
-		(fields_autoplaced yes)
-		(property "Reference" "SAW2"
-			(at 115.57 97.79 0)
-			(show_name no)
-			(do_not_autoplace no)
-			(effects
-				(font
-					(size 1.27 1.27)
-				)
-			)
-		)
-		(property "Value" "B39162B4300F210"
-			(at 115.57 100.33 0)
-			(show_name no)
-			(do_not_autoplace no)
-			(effects
-				(font
-					(size 1.27 1.27)
-				)
-			)
-		)
-		(property "Footprint" "aerolotl_custom:FILTER-SMD_5P-L1.4-W1.1_RSFPXXXXD"
-			(at 115.57 118.11 0)
-			(hide yes)
-			(show_name no)
-			(do_not_autoplace no)
-			(effects
-				(font
-					(size 1.27 1.27)
-				)
-			)
-		)
-		(property "Datasheet" ""
-			(at 115.57 107.95 0)
-			(hide yes)
-			(show_name no)
-			(do_not_autoplace no)
-			(effects
-				(font
-					(size 1.27 1.27)
-				)
-			)
-		)
-		(property "Description" ""
-			(at 115.57 107.95 0)
-			(hide yes)
-			(show_name no)
-			(do_not_autoplace no)
-			(effects
-				(font
-					(size 1.27 1.27)
-				)
-			)
-		)
-		(property "LCSC Part" "C2650962"
-			(at 115.57 120.65 0)
-			(hide yes)
-			(show_name no)
-			(do_not_autoplace no)
-			(effects
-				(font
-					(size 1.27 1.27)
-				)
-			)
-		)
-		(pin "3"
-		)
-		(pin "4"
-		)
-		(pin "5"
-		)
-		(pin "1"
-		)
-		(pin "2"
-		)
-		(instances
-			(project "aerolotl"
-				(path "/3f5bc5ea-feaa-4ed9-b0e0-c918b1fb5754/74e9b1e9-3a21-4de4-9795-bce3dd5092b3"
-					(reference "SAW2")
-					(unit 1)
-				)
-			)
-		)
-	)
-	(symbol
 		(lib_id "Device:C")
 		(at 40.64 180.34 0)
@@
 			)
 		)
-		(property "Footprint" "aerolotl_custom:ADXL345"
+		(property "Footprint" "ADXL345BCCZ-RL7:PQFN80P500X300X100-14N"
 			(at 199.39 57.15 0)
 			(hide yes)
@@
 	)
 	(symbol
-		(lib_id "aerolotl_custom:GP.1575.18.4.A.02")
-		(at 104.14 96.52 0)
-		(unit 1)
-		(body_style 1)
-		(exclude_from_sim no)
-		(in_bom yes)
-		(on_board yes)
-		(in_pos_files yes)
-		(dnp no)
-		(fields_autoplaced yes)
-		(property "Reference" "AE1"
-			(at 107.95 88.8999 0)
-			(show_name no)
-			(do_not_autoplace no)
-			(effects
-				(font
-					(size 1.524 1.524)
-				)
-				(justify left)
-			)
-		)
-		(property "Value" "GP.1575.18.4.A.02"
-			(at 107.95 91.4399 0)
-			(show_name no)
-			(do_not_autoplace no)
-			(effects
-				(font
-					(size 1.524 1.524)
-				)
-				(justify left)
-			)
-		)
-		(property "Footprint" "ANT_GP.1575.18.4.A.02_TAL"
-			(at 104.14 96.52 0)
-			(hide yes)
-			(show_name no)
-			(do_not_autoplace no)
-			(effects
-				(font
-					(size 1.27 1.27)
-					(italic yes)
-				)
-			)
-		)
-		(property "Datasheet" "GP.1575.18.4.A.02"
-			(at 104.14 96.52 0)
-			(hide yes)
-			(show_name no)
-			(do_not_autoplace no)
-			(effects
-				(font
-					(size 1.27 1.27)
-					(italic yes)
-				)
-			)
-		)
-		(property "Description" ""
-			(at 104.14 96.52 0)
-			(hide yes)
-			(show_name no)
-			(do_not_autoplace no)
-			(effects
-				(font
-					(size 1.27 1.27)
-				)
-			)
-		)
-		(pin "1"
-		)
-		(instances
-			(project "aerolotl"
-				(path "/3f5bc5ea-feaa-4ed9-b0e0-c918b1fb5754/74e9b1e9-3a21-4de4-9795-bce3dd5092b3"
-					(reference "AE1")
-					(unit 1)
-				)
-			)
-		)
-	)
-	(symbol
 		(lib_id "RF_GPS:MAX-M10S")
 		(at 66.04 119.38 0)
@@
 	)
 	(symbol
+		(lib_id "aerolotl_custom:GP.1575.18.4.A.02")
+		(at 104.14 96.52 0)
+		(unit 1)
+		(body_style 1)
+		(exclude_from_sim no)
+		(in_bom yes)
+		(on_board yes)
+		(in_pos_files yes)
+		(dnp no)
+		(fields_autoplaced yes)
+		(property "Reference" "AE1"
+			(at 107.95 88.8999 0)
+			(show_name no)
+			(do_not_autoplace no)
+			(effects
+				(font
+					(size 1.524 1.524)
+				)
+				(justify left)
+			)
+		)
+		(property "Value" "GP.1575.18.4.A.02"
+			(at 107.95 91.4399 0)
+			(show_name no)
+			(do_not_autoplace no)
+			(effects
+				(font
+					(size 1.524 1.524)
+				)
+				(justify left)
+			)
+		)
+		(property "Footprint" "aerolotl_custom:ANT_GP.1575.18.4.A.02_TAL"
+			(at 104.14 96.52 0)
+			(hide yes)
+			(show_name no)
+			(do_not_autoplace no)
+			(effects
+				(font
+					(size 1.27 1.27)
+					(italic yes)
+				)
+			)
+		)
+		(property "Datasheet" "GP.1575.18.4.A.02"
+			(at 104.14 96.52 0)
+			(hide yes)
+			(show_name no)
+			(do_not_autoplace no)
+			(effects
+				(font
+					(size 1.27 1.27)
+					(italic yes)
+				)
+			)
+		)
+		(property "Description" ""
+			(at 104.14 96.52 0)
+			(hide yes)
+			(show_name no)
+			(do_not_autoplace no)
+			(effects
+				(font
+					(size 1.27 1.27)
+				)
+			)
+		)
+		(pin "1"
+		)
+		(instances
+			(project "aerolotl"
+				(path "/3f5bc5ea-feaa-4ed9-b0e0-c918b1fb5754/74e9b1e9-3a21-4de4-9795-bce3dd5092b3"
+					(reference "AE1")
+					(unit 1)
+				)
+			)
+		)
+	)
+	(symbol
 		(lib_id "power:+3V3")
 		(at 60.96 91.44 0)
@@
 					(unit 1)
 				)
+			)
+		)
+	)
+	(symbol
+		(lib_id "aerolotl_custom:B39162B4300F210")
+		(at 115.57 107.95 0)
+		(unit 1)
+		(body_style 1)
+		(exclude_from_sim no)
+		(in_bom yes)
+		(on_board yes)
+		(in_pos_files yes)
+		(dnp no)
+		(fields_autoplaced yes)
+		(property "Reference" "SAW1"
+			(at 115.57 97.79 0)
+			(show_name no)
+			(do_not_autoplace no)
+			(effects
+				(font
+					(size 1.27 1.27)
+				)
+			)
+		)
+		(property "Value" "B39162B4300F210"
+			(at 115.57 100.33 0)
+			(show_name no)
+			(do_not_autoplace no)
+			(effects
+				(font
+					(size 1.27 1.27)
+				)
+			)
+		)
+		(property "Footprint" "aerolotl_custom:FILTER-SMD_5P-L1.4-W1.1_RSFPXXXXD"
+			(at 115.57 118.11 0)
+			(hide yes)
+			(show_name no)
+			(do_not_autoplace no)
+			(effects
+				(font
+					(size 1.27 1.27)
+				)
+			)
+		)
+		(property "Datasheet" ""
+			(at 115.57 107.95 0)
+			(hide yes)
+			(show_name no)
+			(do_not_autoplace no)
+			(effects
+				(font
+					(size 1.27 1.27)
+				)
+			)
+		)
+		(property "Description" ""
+			(at 115.57 107.95 0)
+			(hide yes)
+			(show_name no)
+			(do_not_autoplace no)
+			(effects
+				(font
+					(size 1.27 1.27)
+				)
+			)
+		)
+		(property "LCSC Part" "C2650962"
+			(at 115.57 120.65 0)
+			(hide yes)
+			(show_name no)
+			(do_not_autoplace no)
+			(effects
+				(font
+					(size 1.27 1.27)
+				)
+			)
+		)
+		(pin "1"
+		)
+		(pin "2"
+		)
+		(pin "5"
+		)
+		(pin "3"
+		)
+		(pin "4"
+		)
+		(instances
+			(project "aerolotl"
+				(path "/3f5bc5ea-feaa-4ed9-b0e0-c918b1fb5754/74e9b1e9-3a21-4de4-9795-bce3dd5092b3"
+					(reference "SAW1")
+					(unit 1)
+				)
