File: BatteryPCB/sheets/buck_5v.kicad_sch (KiCad schematic)
At the start: 17 parts, among them U1 LMR51430XFDDCR

Commit message: Preserve battery PCB progress and prepare partial JLC assembly files
Parts:
- C1: LCSC (none) -> C49678; MPN CL21B104KBCNNNC -> CC0805KRX7R9BB104; Manufacturer Samsung Electro-Mechanics -> YAGEO
- C4, C5: value 22u / 16V -> 22u / 25V; LCSC (none) -> C45783; MPN CL21A226MOQNNNE -> CL21A226MAQNNNE
Other:
- note added: "so the camera pack stops at about 2.7 V per cell instead of being run flat (U1's own UVLO is 3.6 V)."
- note removed: "so the camera pack stops at about 2.85 V per cell instead of being run flat (U1's own UVLO is 3.6 V)."
Changed lines of the file:
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@@
 		)
 	)
-	(text "so the camera pack stops at about 2.85 V per cell instead of being run flat (U1's own UVLO is 3.6 V)."
+	(text "so the camera pack stops at about 2.7 V per cell instead of being run flat (U1's own UVLO is 3.6 V)."
 		(exclude_from_sim no)
 		(at 25.4 44.45 0)
@@
 			)
 		)
-		(property "Value" "22u / 16V"
+		(property "Value" "22u / 25V"
 			(at 182.88 97.79 0)
 			(show_name no)
@@
 		(pin "2"
 		)
-		(instances
+		    (property "Manufacturer" "Samsung Electro-Mechanics"
+      (at 0 0 0)
+      (effects (font (size 1.27 1.27)) (hide yes))
+    )
+        (property "MPN" "CL21A226MAQNNNE"
+      (at 0 0 0)
+      (effects (font (size 1.27 1.27)) (hide yes))
+    )
+        (property "LCSC" "C45783"
+      (at 0 0 0)
+      (effects (font (size 1.27 1.27)) (hide yes))
+    )
+    (instances
 			(project "battery_pcb"
 				(path "/19ef3a32-de7c-46ee-a850-2420f6d47f94/1914f4ed-278a-4026-a86a-769e5e361ab6"
@@
 			)
 		)
-		(property "Value" "22u / 16V"
+		(property "Value" "22u / 25V"
 			(at 200.66 97.79 0)
 			(show_name no)
@@
 		(pin "2"
 		)
-		(instances
+		    (property "Manufacturer" "Samsung Electro-Mechanics"
+      (at 0 0 0)
+      (effects (font (size 1.27 1.27)) (hide yes))
+    )
+        (property "MPN" "CL21A226MAQNNNE"
+      (at 0 0 0)
+      (effects (font (size 1.27 1.27)) (hide yes))
+    )
+        (property "LCSC" "C45783"
+      (at 0 0 0)
+      (effects (font (size 1.27 1.27)) (hide yes))
+    )
+    (instances
 			(project "battery_pcb"
 				(path "/19ef3a32-de7c-46ee-a850-2420f6d47f94/1914f4ed-278a-4026-a86a-769e5e361ab6"
@@
 		(pin "2"
 		)
-		(instances
+		    (property "Manufacturer" "YAGEO"
+      (at 0 0 0)
+      (effects (font (size 1.27 1.27)) (hide yes))
+    )
+        (property "MPN" "CC0805KRX7R9BB104"
+      (at 0 0 0)
+      (effects (font (size 1.27 1.27)) (hide yes))
+    )
+        (property "LCSC" "C49678"
+      (at 0 0 0)
+      (effects (font (size 1.27 1.27)) (hide yes))
+    )
+    (instances
 			(project "battery_pcb"
 				(path "/19ef3a32-de7c-46ee-a850-2420f6d47f94/1914f4ed-278a-4026-a86a-769e5e361ab6"
