File: BatteryPCB/sheets/supplies.kicad_sch (KiCad schematic)
At the start: 6 parts, among them J5 to COTS altimeter, J6 to SRAD flight computer, SW2 COTS ARM, SW3 SRAD ARM

Commit message: Preserve battery PCB progress and prepare partial JLC assembly files
Parts:
- J5, J6: MPN XT30UPB-F -> XT30UPB-M
Changed lines of the file:
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@@
 		(pin "2"
 		)
-		(instances
+		    (property "MPN" "XT30UPB-M"
+      (at 0 0 0)
+      (effects (font (size 1.27 1.27)) (hide yes))
+    )
+    (instances
 			(project "battery_pcb"
 				(path "/19ef3a32-de7c-46ee-a850-2420f6d47f94/d30d38cc-20d9-4e05-9f85-c70abea8b778"
@@
 		(pin "2"
 		)
-		(instances
+		    (property "MPN" "XT30UPB-M"
+      (at 0 0 0)
+      (effects (font (size 1.27 1.27)) (hide yes))
+    )
+    (instances
 			(project "battery_pcb"
 				(path "/19ef3a32-de7c-46ee-a850-2420f6d47f94/d30d38cc-20d9-4e05-9f85-c70abea8b778"
