File: BatteryPCB/battery_pcb.kicad_pcb (KiCad board)
At the start: 2 copper layers, 145.3 x 142.5 mm, 53 parts, among them J1 ESP32 left, J2 ESP32 right, J3 RunCam Split 4, J5 to COTS altimeter, J6 to SRAD flight computer, SW1 CAM POWER, SW2 COTS ARM, SW3 SRAD ARM, U1 LMR51430XFDDCR

Commit message: Battery PCB v21: R8 1k camera-RX protection, separate drill files
- R8 (camera TX -> ESP32 RX) 100R -> 1k: protects GPIO16 if the
  RunCam's UART turns out to be 5 V.
- Separate PTH/NPTH drill files; tools/make_fab.sh rebuilds fab/.
- README: camera logic-level check, USB + board power is safe (DevKitC
  feeds 5V from USB through a Schottky).
ERC 0 errors, DRC 0 (strict, schematic parity), verify_A all pass.

Co-Authored-By: Claude Opus 5.5 <noreply@anthropic.com>
Parts:
- R8: value 100R -> 1k

Commit message: Battery PCB v22: RunCam standoffs moved out to the upper-left rim
The four SMT camera standoffs (no holes through the board) move from
(-24, 14.75) to (-35.5, -30), about 46 mm from the centre instead of 28,
clear of the ESP32, buck, J3, rod nut, cut-outs and antenna keep-out.
DRC 0 with schematic parity, verify_A all pass. Fab outputs, STEP and
renders regenerated.

Co-Authored-By: Claude Opus 5.5 <noreply@anthropic.com>
Parts:
- moved CAM1 46.2 mm to (114.5, 120.0)
- moved H10 46.2 mm to (127.2, 132.8)
- moved H7 46.2 mm to (101.8, 107.2)
- moved H8 46.2 mm to (127.2, 107.2)
- moved H9 46.2 mm to (101.8, 132.8)
Routing:
- net GND: vias 103 -> 102

Commit message: Battery PCB schematic: ESP32, camera and pack-sense sheets merged; C9/C10 on the buck output
Schematic only: sheets 3-5 become one wired sheet (3. ESP32 + camera), C9/C10 move
to the buck sheet's +5V output, supplies renumbered 6 -> 4. Every connection,
part, value and footprint is unchanged; the board only gets the new sheet paths
and net-name prefixes (tools/sync_from_sch.py). Gerbers and drills are
geometrically identical to v22. DRC 0 with schematic parity.

Co-Authored-By: Claude Opus 5.5 <noreply@anthropic.com>
Connections:
- net /3. Pack voltage sense/VBAT_SENSE renamed /3. ESP32 + camera/VBAT_SENSE
- net /4. ESP32 socket/ESP_RX2 renamed /3. ESP32 + camera/ESP_RX2
- net /4. ESP32 socket/ESP_TX2 renamed /3. ESP32 + camera/ESP_TX2
- net /4. ESP32 socket/L01_3V3 renamed /3. ESP32 + camera/L01_3V3
- net /4. ESP32 socket/L02_EN renamed /3. ESP32 + camera/L02_EN
- net /4. ESP32 socket/L03_IO36 renamed /3. ESP32 + camera/L03_IO36
- net /4. ESP32 socket/L04_IO39 renamed /3. ESP32 + camera/L04_IO39
- net /4. ESP32 socket/L06_IO35 renamed /3. ESP32 + camera/L06_IO35
- net /4. ESP32 socket/L07_IO32 renamed /3. ESP32 + camera/L07_IO32
- net /4. ESP32 socket/L08_IO33 renamed /3. ESP32 + camera/L08_IO33
- net /4. ESP32 socket/L09_IO25 renamed /3. ESP32 + camera/L09_IO25
- net /4. ESP32 socket/L10_IO26 renamed /3. ESP32 + camera/L10_IO26
- net /4. ESP32 socket/L11_IO27 renamed /3. ESP32 + camera/L11_IO27
- net /4. ESP32 socket/L12_IO14 renamed /3. ESP32 + camera/L12_IO14
- net /4. ESP32 socket/L13_IO12 renamed /3. ESP32 + camera/L13_IO12
- net /4. ESP32 socket/L15_IO13 renamed /3. ESP32 + camera/L15_IO13
- net /4. ESP32 socket/L16_IO9 renamed /3. ESP32 + camera/L16_IO9
- net /4. ESP32 socket/L17_IO10 renamed /3. ESP32 + camera/L17_IO10
- net /4. ESP32 socket/L18_IO11 renamed /3. ESP32 + camera/L18_IO11
- net /4. ESP32 socket/LED_A renamed /3. ESP32 + camera/LED_A
- net /4. ESP32 socket/LED_GPIO renamed /3. ESP32 + camera/LED_GPIO
- net /4. ESP32 socket/R02_IO23 renamed /3. ESP32 + camera/R02_IO23
- net /4. ESP32 socket/R03_IO22 renamed /3. ESP32 + camera/R03_IO22
- net /4. ESP32 socket/R04_TX0 renamed /3. ESP32 + camera/R04_TX0
- net /4. ESP32 socket/R05_RX0 renamed /3. ESP32 + camera/R05_RX0
- net /4. ESP32 socket/R06_IO21 renamed /3. ESP32 + camera/R06_IO21
- net /4. ESP32 socket/R08_IO19 renamed /3. ESP32 + camera/R08_IO19
- net /4. ESP32 socket/R09_IO18 renamed /3. ESP32 + camera/R09_IO18
- net /4. ESP32 socket/R10_IO5 renamed /3. ESP32 + camera/R10_IO5
- net /4. ESP32 socket/R13_IO4 renamed /3. ESP32 + camera/R13_IO4
- net /4. ESP32 socket/R14_IO0 renamed /3. ESP32 + camera/R14_IO0
- net /4. ESP32 socket/R16_IO15 renamed /3. ESP32 + camera/R16_IO15
- net /4. ESP32 socket/R17_IO8 renamed /3. ESP32 + camera/R17_IO8
- net /4. ESP32 socket/R18_IO7 renamed /3. ESP32 + camera/R18_IO7
- net /4. ESP32 socket/R19_IO6 renamed /3. ESP32 + camera/R19_IO6
- net /5. RunCam Split 4/CAM_RX renamed /3. ESP32 + camera/CAM_RX
- net /5. RunCam Split 4/CAM_TX renamed /3. ESP32 + camera/CAM_TX
- net /5. RunCam Split 4/CAM_VIDEO renamed /3. ESP32 + camera/CAM_VIDEO
- net /6. COTS / SRAD supplies/COTS_BAT+ renamed /4. COTS / SRAD supplies/COTS_BAT+
- net /6. COTS / SRAD supplies/COTS_BAT- renamed /4. COTS / SRAD supplies/COTS_BAT-
- net /6. COTS / SRAD supplies/COTS_SW renamed /4. COTS / SRAD supplies/COTS_SW
- net /6. COTS / SRAD supplies/SRAD_BAT+ renamed /4. COTS / SRAD supplies/SRAD_BAT+
- net /6. COTS / SRAD supplies/SRAD_BAT- renamed /4. COTS / SRAD supplies/SRAD_BAT-
- net /6. COTS / SRAD supplies/SRAD_SW renamed /4. COTS / SRAD supplies/SRAD_SW

Commit message: Battery PCB: schematic sheets re-saved after cleanup; board net names re-escaped
Same design as 428171c: identical netlist (42 parts, 55 nets, same pins,
values, footprints and MPNs) and identical board geometry. The board only
changes the sheet-name escaping inside net names ("COTS / SRAD" ->
"COTS {slash} SRAD").

Checks on this commit: ERC 0 errors; strict DRC 0 violations, 0 unconnected,
0 schematic parity issues (also with zones refilled); verify_A.py ALL PASS.
New ERC warnings: 16 endpoint_off_grid on the root and COTS/SRAD sheets
(half-grid wire ends and J6 pin 1); connectivity is unaffected.

Co-Authored-By: Claude Opus 5.5 <noreply@anthropic.com>
Connections:
- net /4. COTS / SRAD supplies/COTS_BAT+ renamed /4. COTS / SRAD supplies/COTS_BAT+
- net /4. COTS / SRAD supplies/COTS_BAT- renamed /4. COTS / SRAD supplies/COTS_BAT-
- net /4. COTS / SRAD supplies/COTS_SW renamed /4. COTS / SRAD supplies/COTS_SW
- net /4. COTS / SRAD supplies/SRAD_BAT+ renamed /4. COTS / SRAD supplies/SRAD_BAT+
- net /4. COTS / SRAD supplies/SRAD_BAT- renamed /4. COTS / SRAD supplies/SRAD_BAT-
- net /4. COTS / SRAD supplies/SRAD_SW renamed /4. COTS / SRAD supplies/SRAD_SW

Commit message: Battery PCB v23: review 3 fixes (5 V setpoint, boot cap, GND vias, antenna keep-out)
- R3 13k7 -> 13k (RC0603FR-0713KL, LCSC C137796): 5.22 V nominal,
  5.05-5.39 V worst case, so the RunCam always gets >= 5.0 V.
- C3 moved beside U1; its SW side lands directly on L1's pad (no vias).
- New GND via ~1 mm from U1 pin 1; 5 stitching vias in open GND pour.
- Front antenna no-pour area now matches the back keep-out (48 x 21 mm).
- R10 pad 2 solid to the pour plus a trace to its via.
- fab/ regenerated (BOM, Gerbers, drills, schematic PDF, project zip).

ERC 0 errors; DRC 0 violations / 0 unconnected / 0 parity (also with
zones refilled); verify_A ALL PASS.

Co-Authored-By: Claude Opus 5.5 <noreply@anthropic.com>
Parts:
- R3: value 13k7 1% -> 13k 1%
- moved C3 3.63 mm to (164.3, 139.7), turned to -90 degrees
Routing:
- net /2. Buck to 5 V/SW: track 10.6 -> 4.24 mm, vias 2 -> 0
- net GND: track 24.8 -> 25.6 mm, vias 102 -> 107

Commit message: Battery PCB v24: 3.0 mm pin holes for the camera standoffs (H7-H10)
The Wurth 9774050243R SMT standoff has a 1.4 mm, 2.8 mm-diameter locating
pin on its base; the old _NoHole footprint had nowhere for it, so the
standoffs would have sat 1.4 mm off their pads. H7-H10 now use Wurth's
land pattern with the 3.0 mm non-plated hole (same positions). The pin
stays inside the 1.6 mm board; no front copper within 3.5 mm.

- Front silk line through H8 gets a gap.
- 3 documented DRC exclusions: H9/H10 holes inside BT1/BT2 courtyards,
  BT1 outline silk over H9's hole.
- place_A.py points at the new footprint; old footprint removed.
- fab/ regenerated (NPTH drill now has 4 x 3.0 mm at the standoffs).

ERC 0 errors; DRC 0 active (strict, parity, zones refilled);
verify_A ALL PASS.

Co-Authored-By: Claude Opus 5.5 <noreply@anthropic.com>
Parts:
- H10, H7, H8, H9: footprint battery_pcb:Mounting_Wuerth_WA-SMSI-M2_H5mm_9774050243_NoHole -> battery_pcb:Mounting_Wuerth_WA-SMSI-M2_H5mm_9774050243
Changed lines of the file:
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@@
 		)
 	)
-	(footprint "battery_pcb:Mounting_Wuerth_WA-SMSI-M2_H5mm_9774050243_NoHole"
+	(footprint "battery_pcb:Mounting_Wuerth_WA-SMSI-M2_H5mm_9774050243"
 		(layer "B.Cu")
 		(at 101.75 107.25 180)
-		(descr "Wuerth WA-SMSI M2 x 5 mm SMT standoff 9774050243, land pattern WITHOUT the centre hole (it sits under a battery holder here; use M2 x 5 screws) (https://www.we-online.com/components/products/datasheet/9774050243R.pdf)")
+		(descr "Wuerth WA-SMSI M2 x 5 mm SMT standoff 9774050243R, Wuerth land pattern with the 3.0 mm non-plated hole for the standoff's 1.4 mm pin (https://www.we-online.com/components/products/datasheet/9774050243R.pdf)")
 		(tags "Mounting M2 9774050243")
 		(property "Reference" "H7"
@@
 			)
 		)
+		(pad "" np_thru_hole circle
+			(at 0 0 180)
+			(size 3 3)
+			(drill 3)
+			(layers "*.Cu" "*.Mask")
+		)
 		(pad "" smd custom
 			(at 1.453104 -1.453104 180)
@@
 		)
 	)
-	(footprint "battery_pcb:Mounting_Wuerth_WA-SMSI-M2_H5mm_9774050243_NoHole"
+	(footprint "battery_pcb:Mounting_Wuerth_WA-SMSI-M2_H5mm_9774050243"
 		(layer "B.Cu")
 		(at 101.75 132.75 180)
-		(descr "Wuerth WA-SMSI M2 x 5 mm SMT standoff 9774050243, land pattern WITHOUT the centre hole (it sits under a battery holder here; use M2 x 5 screws) (https://www.we-online.com/components/products/datasheet/9774050243R.pdf)")
+		(descr "Wuerth WA-SMSI M2 x 5 mm SMT standoff 9774050243R, Wuerth land pattern with the 3.0 mm non-plated hole for the standoff's 1.4 mm pin (https://www.we-online.com/components/products/datasheet/9774050243R.pdf)")
 		(tags "Mounting M2 9774050243")
 		(property "Reference" "H9"
@@
 			)
 		)
+		(pad "" np_thru_hole circle
+			(at 0 0 180)
+			(size 3 3)
+			(drill 3)
+			(layers "*.Cu" "*.Mask")
+		)
 		(pad "" smd custom
 			(at 1.453104 -1.453104 180)
@@
 		)
 	)
-	(footprint "battery_pcb:Mounting_Wuerth_WA-SMSI-M2_H5mm_9774050243_NoHole"
+	(footprint "battery_pcb:Mounting_Wuerth_WA-SMSI-M2_H5mm_9774050243"
 		(layer "B.Cu")
 		(at 127.25 132.75 180)
-		(descr "Wuerth WA-SMSI M2 x 5 mm SMT standoff 9774050243, land pattern WITHOUT the centre hole (it sits under a battery holder here; use M2 x 5 screws) (https://www.we-online.com/components/products/datasheet/9774050243R.pdf)")
+		(descr "Wuerth WA-SMSI M2 x 5 mm SMT standoff 9774050243R, Wuerth land pattern with the 3.0 mm non-plated hole for the standoff's 1.4 mm pin (https://www.we-online.com/components/products/datasheet/9774050243R.pdf)")
 		(tags "Mounting M2 9774050243")
 		(property "Reference" "H10"
@@
 			)
 		)
+		(pad "" np_thru_hole circle
+			(at 0 0 180)
+			(size 3 3)
+			(drill 3)
+			(layers "*.Cu" "*.Mask")
+		)
 		(pad "" smd custom
 			(at 1.453104 -1.453104 180)
@@
 		)
 	)
-	(footprint "battery_pcb:Mounting_Wuerth_WA-SMSI-M2_H5mm_9774050243_NoHole"
+	(footprint "battery_pcb:Mounting_Wuerth_WA-SMSI-M2_H5mm_9774050243"
 		(layer "B.Cu")
 		(at 127.25 107.25 180)
-		(descr "Wuerth WA-SMSI M2 x 5 mm SMT standoff 9774050243, land pattern WITHOUT the centre hole (it sits under a battery holder here; use M2 x 5 screws) (https://www.we-online.com/components/products/datasheet/9774050243R.pdf)")
+		(descr "Wuerth WA-SMSI M2 x 5 mm SMT standoff 9774050243R, Wuerth land pattern with the 3.0 mm non-plated hole for the standoff's 1.4 mm pin (https://www.we-online.com/components/products/datasheet/9774050243R.pdf)")
 		(tags "Mounting M2 9774050243")
 		(property "Reference" "H8"
@@
 			)
 		)
+		(pad "" np_thru_hole circle
+			(at 0 0 180)
+			(size 3 3)
+			(drill 3)
+			(layers "*.Cu" "*.Mask")
+		)
 		(pad "" smd custom
 			(at 1.453104 -1.453104 180)
@@
 	(gr_line
 		(start 127.5 81.4)
-		(end 127.5 112.5)
+		(end 127.5 104.75)
 		(stroke
 			(width 0.15)
@@
 		(stroke
 			(width 0.15)
+			(type default)
+		)
+		(layer "F.SilkS")
+	)
+	(gr_line
+		(start 127.5 109.75)
+		(end 127.5 112.5)
+		(stroke
+			(width 0.15)
